File: CPU.sch (KiCad schematic (older format))
At the start: 46 parts, among them CN201 PH-2X4S, CN202 DF11-4DP-2DSA, CN203 DF11-4DP-2DSA, CN204 826646-4, CN205 DF11-8DP-2DSA, CN206 DF11-4DP-2DSA, CN207 DF11-4DP-2DSA, Q201 SSM3K15AFU, Q202 SSM3K15AFU, SW201 SKRPACE010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

Commit message: Rev.01-Add USB-PD CKT
Parts:
- C201, C202, C203, C204, C205, C206, C208, C209, C211, C212, C213: symbol EH-900:C -> EH-900-rescue:C-EH-900
- CN201: symbol EH-900:PIN_HEADER_8PIN -> EH-900-rescue:PIN_HEADER_8PIN-EH-900
- CN202, CN203, CN206, CN207: symbol EH-900:DF11-4DP-2DSA -> EH-900-rescue:DF11-4DP-2DSA-EH-900
- CN204: symbol EH-900:PIN_HEADER_4PIN -> EH-900-rescue:PIN_HEADER_4PIN-EH-900
- CN205: symbol EH-900:DF11-8DP-2DSA -> EH-900-rescue:DF11-8DP-2DSA-EH-900
- D201: symbol main-eagle-import:1SS -> EH-900-rescue:1SS-main-eagle-import
- Q201, Q202: symbol EH-900:Q_NMOS_DGS -> EH-900-rescue:Q_NMOS_DGS-EH-900
- R201, R202, R203, R204, R205, R206, R207, R208, R209, R210, R211, R212, R213, R214, R215, R216, R217: symbol EH-900:R_Thick_1005_Pban -> EH-900-rescue:R_Thick_1005_Pban-EH-900
- SW201: symbol EH-900:SKRPACE010 -> EH-900-rescue:SKRPACE010-EH-900
- U203: symbol EH-900:74VHC125FT -> EH-900-rescue:74VHC125FT-EH-900
- U204: symbol EH-900:TPS79933DDC -> EH-900-rescue:TPS79933DDC-EH-900
Changed lines of the file:
@@
 $EndComp
 $Comp
-L EH-900:R_Thick_1005_Pban R?
+L EH-900-rescue:R_Thick_1005_Pban-EH-900 R?
 U 1 1 6025A0F3
 P 4650 4200
@@
 	4800 3700 4800 4000
 $Comp
-L EH-900:C C?
+L EH-900-rescue:C-EH-900 C?
 U 1 1 6025A126
 P 4750 3400
@@
 $EndComp
 $Comp
-L EH-900:R_Thick_1005_Pban R?
+L EH-900-rescue:R_Thick_1005_Pban-EH-900 R?
 U 1 1 6025A12C
 P 5200 3600
@@
 $EndComp
 $Comp
-L EH-900:C C?
+L EH-900-rescue:C-EH-900 C?
 U 1 1 6025A0E7
 P 3850 4200
@@
 $EndComp
 $Comp
-L EH-900:C C?
+L EH-900-rescue:C-EH-900 C?
 U 1 1 6025A0ED
 P 3850 3700
@@
 SWCLK
 $Comp
-L EH-900:C C?
+L EH-900-rescue:C-EH-900 C?
 U 1 1 6020412C
 P 6400 3000
@@
 Connection ~ 6150 2600
 $Comp
-L EH-900:C C?
+L EH-900-rescue:C-EH-900 C?
 U 1 1 6025A153
 P 6300 2600
@@
 	6950 3200 6950 2400
 $Comp
-L EH-900:Q_NMOS_DGS Q201
+L EH-900-rescue:Q_NMOS_DGS-EH-900 Q201
 U 1 1 60213E66
 P 6400 7950
@@
 $EndComp
 $Comp
-L EH-900:R_Thick_1005_Pban R?
+L EH-900-rescue:R_Thick_1005_Pban-EH-900 R?
 U 1 1 60215E55
 P 6700 8200
@@
 $EndComp
 $Comp
-L EH-900:R_Thick_1005_Pban R?
+L EH-900-rescue:R_Thick_1005_Pban-EH-900 R?
 U 1 1 60216997
 P 7700 7600
@@
 $EndComp
 $Comp
-L EH-900:C C?
+L EH-900-rescue:C-EH-900 C?
 U 1 1 60217CA4
 P 7100 8200
@@
 $EndComp
 $Comp
-L EH-900:R_Thick_1005_Pban R?
+L EH-900-rescue:R_Thick_1005_Pban-EH-900 R?
 U 1 1 602195DA
 P 7400 7950
@@
 	7700 7450 7700 7400
 $Comp
-L EH-900:R_Thick_1005_Pban R?
+L EH-900-rescue:R_Thick_1005_Pban-EH-900 R?
 U 1 1 602271C1
 P 6300 7450
@@
 	5000 3400 5550 3400
 $Comp
-L EH-900:+3V3D #PWR?
+L EH-900-rescue:+3V3D-EH-900 #PWR?
 U 1 1 60244F1E
 P 6950 2400
@@
 $EndComp
 $Comp
-L EH-900:+3V3D #PWR?
+L EH-900-rescue:+3V3D-EH-900 #PWR?
 U 1 1 60245557
 P 6150 2400
@@
 	6150 2500 6150 2400
 $Comp
-L EH-900:Q_NMOS_DGS Q202
+L EH-900-rescue:Q_NMOS_DGS-EH-900 Q202
 U 1 1 602570CC
 P 7400 6550
@@
 $EndComp
 $Comp
-L EH-900:R_Thick_1005_Pban R?
+L EH-900-rescue:R_Thick_1005_Pban-EH-900 R?
 U 1 1 60258ABF
 P 7100 6800
@@
 $EndComp
 $Comp
-L EH-900:R_Thick_1005_Pban R?
+L EH-900-rescue:R_Thick_1005_Pban-EH-900 R?
 U 1 1 60258F72
 P 6850 6550
@@
 	7500 6750 7500 6950
 $Comp
-L EH-900:DF11-4DP-2DSA CN203
+L EH-900-rescue:DF11-4DP-2DSA-EH-900 CN203
 U 1 1 6028A093
 P 8650 6200
@@
 $EndComp
 $Comp
-L EH-900:DF11-4DP-2DSA CN202
+L EH-900-rescue:DF11-4DP-2DSA-EH-900 CN202
 U 1 1 6028B591
 P 4250 6350
@@
 	7500 6150 7500 6350
 $Comp
-L EH-900:R_Thick_1005_Pban R?
+L EH-900-rescue:R_Thick_1005_Pban-EH-900 R?
 U 1 1 602585CD
 P 7650 6150
@@
 $EndComp
 $Comp
-L EH-900:+5VD #PWR0232
+L EH-900-rescue:+5VD-EH-900 #PWR0232
 U 1 1 602F9943
 P 7700 7400
@@
 $EndComp
 $Comp
-L EH-900:+3V3D #PWR?
+L EH-900-rescue:+3V3D-EH-900 #PWR?
 U 1 1 602FAAA4
 P 6300 7200
@@
 $EndComp
 $Comp
-L EH-900:+5VD #PWR0233
+L EH-900-rescue:+5VD-EH-900 #PWR0233
 U 1 1 602FB31C
 P 8300 6050
@@
 	4350 6500 4450 6500
 $Comp
-L EH-900:+3V3D #PWR?
+L EH-900-rescue:+3V3D-EH-900 #PWR?
 U 1 1 6033108A
 P 4400 6200
@@
 I2C1_SDA
 $Comp
-L EH-900:PIN_HEADER_8PIN CN201
+L EH-900-rescue:PIN_HEADER_8PIN-EH-900 CN201
 U 1 1 60358428
 P 4300 7500
@@
 $EndComp
 $Comp
-L EH-900:+3V3D #PWR?
+L EH-900-rescue:+3V3D-EH-900 #PWR?
 U 1 1 6035EEFD
 P 4750 7100
@@
 	4400 7100 4750 7100
 $Comp
-L EH-900:R_Thick_1005_Pban R?
+L EH-900-rescue:R_Thick_1005_Pban-EH-900 R?
 U 1 1 601A2F28
 P 5000 6050
@@
 $EndComp
 $Comp
-L EH-900:R_Thick_1005_Pban R?
+L EH-900-rescue:R_Thick_1005_Pban-EH-900 R?
 U 1 1 601B234B
 P 5300 6050
@@
 $EndComp
 $Comp
-L EH-900:+3V3D #PWR?
+L EH-900-rescue:+3V3D-EH-900 #PWR?
 U 1 1 601B2588
 P 5000 5900
@@
 $EndComp
 $Comp
-L EH-900:+3V3D #PWR?
+L EH-900-rescue:+3V3D-EH-900 #PWR?
 U 1 1 601B2DF5
 P 5300 5900
@@
 	6700 7950 7100 7950
 $Comp
-L EH-900:C C?
+L EH-900-rescue:C-EH-900 C?
 U 1 1 6025A159
 P 5900 2600
@@
 Connection ~ 5000 3000
 $Comp
-L EH-900:PIN_HEADER_4PIN CN204
+L EH-900-rescue:PIN_HEADER_4PIN-EH-900 CN204
 U 1 1 60210509
 P 4300 8700
@@
 I2C1_SCL
 $Comp
-L EH-900:+3V3D #PWR?
+L EH-900-rescue:+3V3D-EH-900 #PWR?
 U 1 1 6021C3E3
 P 5100 8500
@@
 	4500 8600 4500 8650
 $Comp
-L EH-900:DF11-8DP-2DSA CN205
+L EH-900-rescue:DF11-8DP-2DSA-EH-900 CN205
 U 1 1 60273D50
 P 8750 4550
@@
 $EndComp
 $Comp
-L EH-900:+5VD #PWR0114
+L EH-900-rescue:+5VD-EH-900 #PWR0114
 U 1 1 6027A50E
 P 8500 4150
@@
 RESET
 $Comp
-L EH-900:DF11-4DP-2DSA CN206
+L EH-900-rescue:DF11-4DP-2DSA-EH-900 CN206
 U 1 1 603264AD
 P 12250 6600
@@
 $EndComp
 $Comp
-L EH-900:+5VD #PWR0119
+L EH-900-rescue:+5VD-EH-900 #PWR0119
 U 1 1 60397E28
 P 13300 6300
@@
 DC5V in
 $Comp
-L EH-900:TPS79933DDC U204
+L EH-900-rescue:TPS79933DDC-EH-900 U204
 U 1 1 601D16FA
 P 11050 4400
@@
 $EndComp
 $Comp
-L EH-900:C C?
+L EH-900-rescue:C-EH-900 C?
 U 1 1 601D3A99
 P 10150 4650
@@
 	10150 4800 10150 4900
 $Comp
-L EH-900:C C?
+L EH-900-rescue:C-EH-900 C?
 U 1 1 601FDE55
 P 12000 4650
@@
 $EndComp
 $Comp
-L EH-900:C C?
+L EH-900-rescue:C-EH-900 C?
 U 1 1 60218D90
 P 11600 4750
@@
 	12000 4800 12000 4900
 $Comp
-L EH-900:+3V3D #PWR?
+L EH-900-rescue:+3V3D-EH-900 #PWR?
 U 1 1 6022C346
 P 12000 4400
@@
 Connection ~ 12000 4400
 $Comp
-L EH-900:+5VD #PWR0128
+L EH-900-rescue:+5VD-EH-900 #PWR0128
 U 1 1 601E04E1
 P 10150 4400
@@
 	13300 6450 13300 6650
 $Comp
-L EH-900:74VHC125FT U203
+L EH-900-rescue:74VHC125FT-EH-900 U203
 U 1 1 602B2CB5
 P 10800 2750
@@
 $EndComp
 $Comp
-L EH-900:74VHC125FT U203
+L EH-900-rescue:74VHC125FT-EH-900 U203
 U 2 1 602B943F
 P 9950 6850
@@
 $EndComp
 $Comp
-L EH-900:74VHC125FT U203
+L EH-900-rescue:74VHC125FT-EH-900 U203
 U 3 1 602BA4C0
 P 10750 6850
@@
 $EndComp
 $Comp
-L EH-900:74VHC125FT U203
+L EH-900-rescue:74VHC125FT-EH-900 U203
 U 4 1 602BB64F
 P 10400 3200
@@
 $EndComp
 $Comp
-L EH-900:74VHC125FT U203
+L EH-900-rescue:74VHC125FT-EH-900 U203
 U 5 1 602BC87E
 P 13100 4650
@@
 $EndComp
 $Comp
-L EH-900:R_Thick_1005_Pban R?
+L EH-900-rescue:R_Thick_1005_Pban-EH-900 R?
 U 1 1 6025B66D
 P 9500 7050
@@
 $EndComp
 $Comp
-L EH-900:R_Thick_1005_Pban R?
+L EH-900-rescue:R_Thick_1005_Pban-EH-900 R?
 U 1 1 6025C411
 P 10350 7050
@@
 $EndComp
 $Comp
-L EH-900:+3V3D #PWR?
+L EH-900-rescue:+3V3D-EH-900 #PWR?
 U 1 1 602A0B67
 P 13100 3800
@@
 $EndComp
 $Comp
-L EH-900:+5VD #PWR0133
+L EH-900-rescue:+5VD-EH-900 #PWR0133
 U 1 1 602A195A
 P 12800 3800
@@
 $EndComp
 $Comp
-L EH-900:R_Thick_1005_Pban R?
+L EH-900-rescue:R_Thick_1005_Pban-EH-900 R?
 U 1 1 602A2A7B
 P 12800 3950
@@
 $EndComp
 $Comp
-L EH-900:R_Thick_1005_Pban R?
+L EH-900-rescue:R_Thick_1005_Pban-EH-900 R?
 U 1 1 602A3465
 P 13100 3950
@@
 	13100 4250 13100 4300
 $Comp
-L EH-900:C C?
+L EH-900-rescue:C-EH-900 C?
 U 1 1 602B62FF
 P 12800 4650
@@
 	12800 4800 12800 4950
 $Comp
-L EH-900:DF11-4DP-2DSA CN207
+L EH-900-rescue:DF11-4DP-2DSA-EH-900 CN207
 U 1 1 60346642
 P 12100 3150
@@
 $EndComp
 $Comp
-L EH-900:+5VD #PWR0135
+L EH-900-rescue:+5VD-EH-900 #PWR0135
 U 1 1 603483E1
 P 11850 2750
@@
 CONSOLE
 $Comp
-L EH-900:R_Thick_1005_Pban R?
+L EH-900-rescue:R_Thick_1005_Pban-EH-900 R?
 U 1 1 603BB56B
 P 11350 3200
@@
 	11500 3200 12000 3200
 $Comp
-L EH-900:R_Thick_1005_Pban R?
+L EH-900-rescue:R_Thick_1005_Pban-EH-900 R?
 U 1 1 603BC7FD
 P 11500 2750
@@
 	11750 3100 12000 3100
 $Comp
-L main-eagle-import:1SS D201
+L EH-900-rescue:1SS-main-eagle-import D201
 U 1 1 603E238D
 P 11300 2300
@@
 $EndComp
 $Comp
-L EH-900:+5VD #PWR0137
+L EH-900-rescue:+5VD-EH-900 #PWR0137
 U 1 1 603E6368
 P 11100 2300
@@
 	11300 2750 11350 2750
 $Comp
-L EH-900:SKRPACE010 SW201
+L EH-900-rescue:SKRPACE010-EH-900 SW201
 U 1 1 602D89E5
 P 4650 2900
