File: EH-900.kicad_pcb (KiCad board)
At the start: 2 copper layers, 126 x 130 mm, 160 parts, among them CN201 PH-2X4S, CN202 DF11-4DP-2DSA, CN203 DF11-4DP-2DSA, CN204 826646-4, CN205 DF11-8DP-2DSA, CN206 DF11-4DP-2DSA, CN207 DF11-4DP-2DSA, CN301 DF11-4DS-2C, CN302 DF11-4DS-2C, CN304 DF11-4DP-2DSA, CN401 DF11-4DP-2DSA, CN402 DF11-8DP-2DSA, CN403 5267-06A, J301 UJC-HP-3-SMT-TR, Q201 SSM3K15AFU, Q202 SSM3K15AFU, Q301 IRF9362, Q302 Q_NMOS_DGS, Q401 SSM3K15AFU, SW201 SKRPACE010, U201 STM32F303K8T6, U203 74VHCT125AFT, U204 TPS79933DDC, U301 CYPD3177-24LQXQ, U302 OKL-T_3-W12N-C, U401 OPA2344EA, U402 MB85RC256V, U403 ADS1115IDGS, U404 TPS79933DDC, U405 DAC80501ZDGS, U406 MCP4725A0T, U407 MCP23008-xSS, U408 LTC6102CMS8, U409 LT3922, Y201 FA238-16MHz

Commit message: artwork was completed
Parts:
- CN301: value DF11-4DS-2C -> DF11-4DP-2DSA
- CN302: value DF11-4DS-2C -> DF11-6DP-2DSA; footprint Connector_Hirose:Hirose_DF11-4DP-2DSA_2x02_P2.00mm_Vertical -> Connector_Hirose:Hirose_DF11-6DP-2DSA_2x03_P2.00mm_Vertical
- J301: footprint UJC-HP-3-SMT-TR:CUI_UJC-HP-3-SMT-TR -> EH-900:CUI_UJC-HP-3-SMT-TR
- U302: footprint SamacSys_Parts:OKLT3W12PC -> EH-900:OKLT3W12PC
- moved CN304 0.36 mm to (202.1, 54.4)
- moved CN302 0.25 mm to (181.8, 52.6)
- moved CN301 0.13 mm to (153.8, 53.1)
Connections:
- R317 pad 1: Net-(CN303-Pad1) -> Net-(CN302-Pad5)
- R318 pad 2: Net-(CN303-Pad1) -> Net-(CN302-Pad5)
Routing:
- net Net-(CN302-Pad5): track 0.00 -> 31.4 mm, vias 0 -> 1
- net Net-(CN303-Pad1): track 1.85 -> 0.00 mm
- net GNDA: vias 21 -> 22
- net (no net): vias 1 -> 0
- removed copper zone on B.Cu, net Net-(C214-Pad1)

Commit message: Rev.01-Add USB-PD CKT
Parts:
- R317, R318, R319, R320: footprint Resistor_SMD:R_0402_1005Metric_Pad0.72x0.64mm_HandSolder -> Resistor_SMD:R_0603_1608Metric_Pad0.98x0.95mm_HandSolder
- R402, R404: value 10k -> 100k/THICK
- moved R317 1.02 mm to (181.0, 69.4)
- moved R320 0.76 mm to (190.9, 83.6)
- moved R314 0.57 mm to (158.2, 69.4)
- moved R310 0.25 mm to (157.2, 71.1)
- moved R311 0.25 mm to (154.6, 71.1)
Connections:
- net Net-(J301-PadA5) renamed /USB PD Power Supply/CC1
- net Net-(J301-PadB5) renamed /USB PD Power Supply/CC2
- U301 pad 11: Net-(U301-Pad11) -> Net-(C307-Pad1)
Routing:
- net Net-(C307-Pad1): track 0.00 -> 22.3 mm, vias 0 -> 2
- net +3V3A: track 103.0 -> 110.7 mm
- net +5VA: track 49.0 -> 44.8 mm
- net /Measurement Unit/SDA_MU: track 73.3 -> 70.0 mm
- net Net-(D301-Pad2): track 20.3 -> 17.0 mm
- net GNDD: track 37.1 -> 35.8 mm, vias 11 -> 26
- net /Measurement Unit/SCL_MU: track 66.5 -> 65.3 mm
- net Net-(C302-Pad1): track 11.7 -> 10.8 mm, vias 6 -> 0
- net Net-(C212-Pad1): track 3.08 -> 2.21 mm
- net Net-(CN302-Pad5): track 31.4 -> 30.7 mm
- net Net-(C308-Pad1): track 7.41 -> 8.13 mm
- net Net-(C312-Pad1): track 12.3 -> 12.8 mm
- net Net-(R310-Pad2): track 12.7 -> 13.2 mm
- net Net-(D301-Pad1): vias 0 -> 7
- net GNDA: vias 22 -> 31
- added copper zone on B.Cu, net Net-(D301-Pad1)
Other:
- board size 126 x 130 mm -> 105 x 73 mm
- net class AnalogSig removed
- net class Default removed
- net class Power removed
