File: USB_C_PD_DCDC_5V6A.sch (KiCad schematic (older format))
At the start: 43 parts, among them CN301 DF11-4DS-2C, CN302 DF11-4DS-2C, CN303 DF11-4DP-2DSA, CN304 DF11-4DP-2DSA, J301 UJC-HP-3-SMT-TR, Q301 IRF9362, Q302 Q_NMOS_DGS, U301 CYPD3177-24LQXQ, U302 OKL-T_3-W12N-C

Commit message: artwork was completed
Parts:
- removed CN301, CN302: DF11-4DS-2C, Connector_Hirose:Hirose_DF11-4DP-2DSA_2x02_P2.00mm_Vertical, symbol EH-900:DF11-4DS-2C
- removed CN303: DF11-4DP-2DSA, Connector_Hirose:Hirose_DF11-4DP-2DSA_2x02_P2.00mm_Vertical, symbol EH-900:DF11-4DP-2DSA
- added CN301: DF11-4DP-2DSA, Connector_Hirose:Hirose_DF11-4DP-2DSA_2x02_P2.00mm_Vertical, symbol EH-900:DF11-4DP-2DSA
- added CN302: DF11-6DP-2DSA, Connector_Hirose:Hirose_DF11-6DP-2DSA_2x03_P2.00mm_Vertical, symbol main-eagle-import:DF11-6DP-2DSA
- J301: footprint CUI_UJC-HP-3-SMT-TR -> EH-900:CUI_UJC-HP-3-SMT-TR
- U302: footprint OKLT3W12PC -> EH-900:OKLT3W12PC
Connections:
- wire segments 162 -> 164
Other:
- note added: "5-6 SHORT=ON\n"
- note removed: "1-2 SHORT=ON\n"
Changed lines of the file:
@@
 F 0 "J301" H 2693 3267 50  0000 C CNN
 F 1 "UJC-HP-3-SMT-TR" H 2693 3176 50  0000 C CNN
-F 2 "CUI_UJC-HP-3-SMT-TR" H 2800 3500 50  0001 L BNN
+F 2 "EH-900:CUI_UJC-HP-3-SMT-TR" H 2800 3500 50  0001 L BNN
 F 3 "https://jp.cuidevices.com/product/resource/ujc-hp-3-smt-tr.pdf" H 2800 2800 50  0001 L BNN
 F 4 "Manufacturer recommendations" H 2800 3150 50  0001 L BNN "STANDARD"
@@
 F 0 "U302" H 13575 2865 50  0000 C CNN
 F 1 "OKL-T_3-W12N-C" H 13575 2774 50  0000 C CNN
-F 2 "OKLT3W12PC" H 12850 3600 50  0001 L CNN
+F 2 "EH-900:OKLT3W12PC" H 12850 3600 50  0001 L CNN
 F 3 "https://www.mouser.jp/datasheet/2/281/okl-t3-w12-56459.pdf" H 14500 2600 50  0001 L CNN
 F 4 "Module DC-DC 12VIN 1-OUT 0.591V to 5.5V 3A 15W 11-Pin ILGA T/R" H 12850 3400 50  0001 L CNN "Description"
@@
 $EndComp
 $Comp
-L EH-900:DF11-4DP-2DSA CN303
-U 1 1 62481B35
-P 12000 3600
-F 0 "CN303" V 11950 3850 51  0000 L CNN
-F 1 "DF11-4DP-2DSA" V 12200 3200 51  0000 L CNN
-F 2 "Connector_Hirose:Hirose_DF11-4DP-2DSA_2x02_P2.00mm_Vertical" H 12000 3600 50  0001 C CNN
-F 3 "" H 12000 3600 50  0001 C CNN
-	1    12000 3600
-	-1   0    0    -1
-$EndComp
-$Comp
 L EH-900:DF11-4DP-2DSA CN304
 U 1 1 6248490E
@@
 	1    14900 2750
 	1    0    0    -1
-$EndComp
-$Comp
-L EH-900:DF11-4DS-2C CN302
-U 1 1 6249A929
-P 10050 2750
-F 0 "CN302" H 10067 3128 51  0000 C CNN
-F 1 "DF11-4DS-2C" H 10067 3035 51  0000 C CNN
-F 2 "Connector_Hirose:Hirose_DF11-4DP-2DSA_2x02_P2.00mm_Vertical" H 10050 2750 50  0001 C CNN
-F 3 "https://www.hirose.com/ja/product/document?clcode=&productname=&series=DF11&documenttype=Catalog&lang=ja&documentid=D31688_ja" H 10050 2750 50  0001 C CNN
-	1    10050 2750
-	-1   0    0    -1
 $EndComp
 $Comp
@@
 Wire Wire Line
 	12200 2950 12200 3450
-Wire Wire Line
-	12200 3450 12100 3450
 $Comp
 L power:GNDD #PWR0317
 U 1 1 624E4173
-P 12200 3900
-F 0 "#PWR0317" H 12200 3650 50  0001 C CNN
-F 1 "GNDD" H 12204 3745 50  0000 C CNN
-F 2 "" H 12200 3900 50  0001 C CNN
-F 3 "" H 12200 3900 50  0001 C CNN
-	1    12200 3900
-	1    0    0    -1
-$EndComp
-Wire Wire Line
-	12100 3550 12200 3550
-Wire Wire Line
-	12200 3550 12200 3900
-Wire Wire Line
-	10150 2800 10350 2800
+P 9950 3350
+F 0 "#PWR0317" H 9950 3100 50  0001 C CNN
+F 1 "GNDD" H 9954 3195 50  0000 C CNN
+F 2 "" H 9950 3350 50  0001 C CNN
+F 3 "" H 9950 3350 50  0001 C CNN
+	1    9950 3350
+	1    0    0    -1
+$EndComp
+Wire Wire Line
+	9850 3100 9950 3100
+Wire Wire Line
+	9950 3100 9950 3350
+Wire Wire Line
+	9850 2800 10350 2800
 Wire Wire Line
 	10350 2800 10350 2900
 Wire Wire Line
-	10150 2900 10350 2900
+	9850 2900 10350 2900
 Connection ~ 10350 2900
 Wire Wire Line
@@
 Text Notes 14700 2250 0    100  ~ 0
 5V OUT\n
-Text Notes 10150 2250 2    100  ~ 0
+Text Notes 9800 2350 2    100  ~ 0
 9V IN\n
 $Comp
@@
 	14500 3400 14500 3550
 Wire Wire Line
-	10150 2700 10350 2700
-Wire Wire Line
-	10350 2600 10150 2600
+	9850 2700 10350 2700
+Wire Wire Line
+	10350 2600 9850 2600
 Connection ~ 10350 2600
 Wire Wire Line
@@
 Text Notes 13900 4400 2    100  ~ 0
 Vout=5V\n\n
-Text Notes 11650 3550 2    100  ~ 0
-1-2 SHORT=ON\n
-$Comp
-L EH-900:DF11-4DS-2C CN301
-U 1 1 6251080A
+Text Notes 10550 3850 2    100  ~ 0
+5-6 SHORT=ON\n
+$Comp
+L main-eagle-import:DF11-6DP-2DSA CN302
+U 1 1 62616009
+P 9750 2900
+F 0 "CN302" H 9788 3377 42  0000 C CNN
+F 1 "DF11-6DP-2DSA" H 9788 3298 42  0000 C CNN
+F 2 "Connector_Hirose:Hirose_DF11-6DP-2DSA_2x03_P2.00mm_Vertical" H 9750 2900 50  0001 C CNN
+F 3 "" H 9750 2900 50  0001 C CNN
+	1    9750 2900
+	-1   0    0    -1
+$EndComp
+Wire Wire Line
+	9850 3000 10100 3000
+Wire Wire Line
+	10100 3000 10100 3450
+Wire Wire Line
+	10100 3450 12200 3450
+$Comp
+L EH-900:DF11-4DP-2DSA CN301
+U 1 1 626593A7
 P 8750 2750
-F 0 "CN301" H 8767 3128 51  0000 C CNN
-F 1 "DF11-4DS-2C" H 8767 3035 51  0000 C CNN
+F 0 "CN301" H 8500 3100 51  0000 L CNN
+F 1 "DF11-4DP-2DSA" H 8500 3000 51  0000 L CNN
 F 2 "Connector_Hirose:Hirose_DF11-4DP-2DSA_2x02_P2.00mm_Vertical" H 8750 2750 50  0001 C CNN
-F 3 "https://www.hirose.com/ja/product/document?clcode=&productname=&series=DF11&documenttype=Catalog&lang=ja&documentid=D31688_ja" H 8750 2750 50  0001 C CNN
+F 3 "" H 8750 2750 50  0001 C CNN
 	1    8750 2750
 	1    0    0    -1

Commit message: organaize symbol libs
Parts:
- U302: symbol EH-900-rescue:OKL-T_3-W12N-C-SamacSys_Parts -> SamacSys_Parts:OKL-T_3-W12N-C
Changed lines of the file:
@@
 $EndComp
 $Comp
-L EH-900-rescue:OKL-T_3-W12N-C-SamacSys_Parts U302
+L SamacSys_Parts:OKL-T_3-W12N-C U302
 U 1 1 624770BC
 P 12350 2600

Commit message: Rev.01-Add USB-PD CKT
Parts:
- C301, C302, C303, C304, C305, C306, C307, C308, C309, C310, C311, C312: symbol EH-900:C -> EH-900-rescue:C-EH-900
- CN301, CN304: symbol EH-900:DF11-4DP-2DSA -> EH-900-rescue:DF11-4DP-2DSA-EH-900
- CN302: symbol main-eagle-import:DF11-6DP-2DSA -> EH-900-rescue:DF11-6DP-2DSA-main-eagle-import
- J301: symbol UJC-HP-3-SMT-TR:UJC-HP-3-SMT-TR -> EH-900-rescue:UJC-HP-3-SMT-TR-UJC-HP-3-SMT-TR
- Q302: symbol EH-900:Q_NMOS_DGS -> EH-900-rescue:Q_NMOS_DGS-EH-900
- R301, R302, R303, R304, R305, R306, R307, R308, R309, R310, R311, R312, R313, R314, R315, R316: symbol EH-900:R -> EH-900-rescue:R-EH-900
- R317, R318, R319, R320: footprint Resistor_SMD:R_0402_1005Metric_Pad0.72x0.64mm_HandSolder -> Resistor_SMD:R_0603_1608Metric_Pad0.98x0.95mm_HandSolder; symbol EH-900:R -> EH-900-rescue:R-EH-900
- U301: symbol EH-900:CYPD3177-24LQXQ -> EH-900-rescue:CYPD3177-24LQXQ-EH-900
- U302: symbol SamacSys_Parts:OKL-T_3-W12N-C -> EH-900-rescue:OKL-T_3-W12N-C-SamacSys_Parts
Connections:
- net CC1: now reaches J301.A5 (CC1), U301.15 (CC1)
- net CC2: now reaches J301.B5 (CC2), U301.14 (CC2)
- net at U301.11 (VDC_OUT): now also C307.1, CN301.1, CN301.2, Q301.5 (D), Q301.6 (G)
Other:
- note added: "5V/3A OUT\n"
- note removed: "5V OUT\n"
Changed lines of the file:
@@
 for detail:\nhttps://www.notion.so/df9a5d5f49224e88b38ea9e8d9003776
 $Comp
-L UJC-HP-3-SMT-TR:UJC-HP-3-SMT-TR J301
+L EH-900-rescue:UJC-HP-3-SMT-TR-UJC-HP-3-SMT-TR J301
 U 1 1 622F77E3
 P 2800 2800
@@
 $EndComp
 $Comp
-L EH-900:CYPD3177-24LQXQ U301
+L EH-900-rescue:CYPD3177-24LQXQ-EH-900 U301
 U 1 1 6230BE9A
 P 5150 5150
@@
 F 1 "CYPD3177-24LQXQ" H 6150 6100 50  0000 C CNN
 F 2 "Package_DFN_QFN:QFN-24-1EP_4x4mm_P0.5mm_EP2.6x2.6mm" H 4850 5450 50  0001 C CNN
-F 3 "" H 4850 5450 50  0001 C CNN
+F 3 "https://www.mouser.jp/datasheet/2/100/CYPR_S_A0012903526_1-2541381.pdf" H 4850 5450 50  0001 C CNN
 	1    5150 5150
 	1    0    0    -1
@@
 	4000 4900 4350 4900
 $Comp
-L EH-900:C C306
+L EH-900-rescue:C-EH-900 C306
 U 1 1 6231B69B
 P 5800 6350
@@
 $EndComp
 $Comp
-L EH-900:C C303
+L EH-900-rescue:C-EH-900 C303
 U 1 1 6231F4FC
 P 4650 7000
@@
 $EndComp
 $Comp
-L EH-900:C C304
+L EH-900-rescue:C-EH-900 C304
 U 1 1 623208EC
 P 5050 7000
@@
 $EndComp
 $Comp
-L EH-900:C C301
+L EH-900-rescue:C-EH-900 C301
 U 1 1 6234060D
 P 4250 7000
@@
 Connection ~ 4250 6750
 $Comp
-L EH-900:R R308
+L EH-900-rescue:R-EH-900 R308
 U 1 1 62384E0A
 P 3800 5050
@@
 $EndComp
 $Comp
-L EH-900:R R309
+L EH-900-rescue:R-EH-900 R309
 U 1 1 62386487
 P 3800 6000
@@
 $EndComp
 $Comp
-L EH-900:R R306
+L EH-900-rescue:R-EH-900 R306
 U 1 1 62389DF3
 P 3500 5050
@@
 $EndComp
 $Comp
-L EH-900:R R307
+L EH-900-rescue:R-EH-900 R307
 U 1 1 6238A4D8
 P 3500 6000
@@
 	3100 5600 4350 5600
 $Comp
-L EH-900:R R303
+L EH-900-rescue:R-EH-900 R303
 U 1 1 623A83DD
 P 3100 5050
@@
 $EndComp
 $Comp
-L EH-900:R R301
+L EH-900-rescue:R-EH-900 R301
 U 1 1 623A91FA
 P 2800 5050
@@
 $EndComp
 $Comp
-L EH-900:R R304
+L EH-900-rescue:R-EH-900 R304
 U 1 1 623A9D3F
 P 3100 6000
@@
 $EndComp
 $Comp
-L EH-900:R R302
+L EH-900-rescue:R-EH-900 R302
 U 1 1 623AA5AC
 P 2800 6000
@@
 PD_3V3
 $Comp
-L EH-900:Q_NMOS_DGS Q302
+L EH-900-rescue:Q_NMOS_DGS-EH-900 Q302
 U 1 1 623E739B
 P 6950 4800
@@
 $EndComp
 $Comp
-L EH-900:R R315
+L EH-900-rescue:R-EH-900 R315
 U 1 1 623E966E
 P 6700 5250
@@
 	6300 5400 6300 5600
 $Comp
-L EH-900:R R312
+L EH-900-rescue:R-EH-900 R312
 U 1 1 623CCBC1
 P 6300 5250
@@
 $EndComp
 $Comp
-L EH-900:R R316
+L EH-900-rescue:R-EH-900 R316
 U 1 1 62409ABD
 P 7300 4450
@@
 $EndComp
 $Comp
-L EH-900:R R311
+L EH-900-rescue:R-EH-900 R311
 U 1 1 62482D33
 P 5150 2850
@@
 $EndComp
 $Comp
-L EH-900:C C305
+L EH-900-rescue:C-EH-900 C305
 U 1 1 62483B31
 P 5500 2850
@@
 $EndComp
 $Comp
-L EH-900:C C302
+L EH-900-rescue:C-EH-900 C302
 U 1 1 62485E53
 P 4350 3200
@@
 $EndComp
 $Comp
-L EH-900:R R314
+L EH-900-rescue:R-EH-900 R314
 U 1 1 624892AA
 P 6650 3350
@@
 $EndComp
 $Comp
-L EH-900:R R310
+L EH-900-rescue:R-EH-900 R310
 U 1 1 6248A38F
 P 5000 4000
@@
 $EndComp
 $Comp
-L EH-900:R R313
+L EH-900-rescue:R-EH-900 R313
 U 1 1 6248AB84
 P 6500 2850
@@
 	6650 3100 6500 3100
 $Comp
-L EH-900:C C307
+L EH-900-rescue:C-EH-900 C307
 U 1 1 624E7484
 P 7600 2850
@@
 	3300 2600 4350 2600
 Wire Wire Line
-	7600 2600 8550 2600
+	7600 2600 8150 2600
 $Comp
 L Device:LED D302
@@
 	8550 2900 8550 3100
 $Comp
-L EH-900:R R305
+L EH-900-rescue:R-EH-900 R305
 U 1 1 624473AB
 P 3450 3300
@@
 $EndComp
 $Comp
-L SamacSys_Parts:OKL-T_3-W12N-C U302
+L EH-900-rescue:OKL-T_3-W12N-C-SamacSys_Parts U302
 U 1 1 624770BC
 P 12350 2600
@@
 $EndComp
 $Comp
-L EH-900:R R319
+L EH-900-rescue:R-EH-900 R319
 U 1 1 6247B396
 P 13050 3600
 F 0 "R319" V 12950 3500 50  0000 L CNN
 F 1 "1k/THICK" V 13150 3500 50  0000 L CNN
-F 2 "Resistor_SMD:R_0402_1005Metric_Pad0.72x0.64mm_HandSolder" V 12980 3600 50  0001 C CNN
+F 2 "Resistor_SMD:R_0603_1608Metric_Pad0.98x0.95mm_HandSolder" V 12980 3600 50  0001 C CNN
 F 3 "~" H 13050 3600 50  0001 C CNN
 F 4 "SMD" H 13050 3600 50  0001 C CNN "Soldering"
@@
 $EndComp
 $Comp
-L EH-900:R R320
+L EH-900-rescue:R-EH-900 R320
 U 1 1 6247CF33
 P 13050 4050
 F 0 "R320" V 12950 3950 50  0000 L CNN
 F 1 "330/THICK" V 13150 3950 50  0000 L CNN
-F 2 "Resistor_SMD:R_0402_1005Metric_Pad0.72x0.64mm_HandSolder" V 12980 4050 50  0001 C CNN
+F 2 "Resistor_SMD:R_0603_1608Metric_Pad0.98x0.95mm_HandSolder" V 12980 4050 50  0001 C CNN
 F 3 "~" H 13050 4050 50  0001 C CNN
 F 4 "SMD" H 13050 4050 50  0001 C CNN "Soldering"
@@
 $EndComp
 $Comp
-L EH-900:DF11-4DP-2DSA CN304
+L EH-900-rescue:DF11-4DP-2DSA-EH-900 CN304
 U 1 1 6248490E
 P 14900 2750
@@
 $EndComp
 $Comp
-L EH-900:C C309
+L EH-900-rescue:C-EH-900 C309
 U 1 1 624A07F9
 P 11050 2850
@@
 $EndComp
 $Comp
-L EH-900:C C310
+L EH-900-rescue:C-EH-900 C310
 U 1 1 624A2C29
 P 11450 2850
@@
 $EndComp
 $Comp
-L EH-900:C C312
+L EH-900-rescue:C-EH-900 C312
 U 1 1 624A437E
 P 14500 3250
@@
 $EndComp
 $Comp
-L EH-900:C C308
+L EH-900-rescue:C-EH-900 C308
 U 1 1 624A5AA6
 P 10650 2850
@@
 	13550 3400 13550 3550
 $Comp
-L EH-900:R R317
+L EH-900-rescue:R-EH-900 R317
 U 1 1 625296AD
 P 11950 2950
 F 0 "R317" V 11850 2850 50  0000 L CNN
 F 1 "20k/THICK" V 12050 2850 50  0000 L CNN
-F 2 "Resistor_SMD:R_0402_1005Metric_Pad0.72x0.64mm_HandSolder" V 11880 2950 50  0001 C CNN
+F 2 "Resistor_SMD:R_0603_1608Metric_Pad0.98x0.95mm_HandSolder" V 11880 2950 50  0001 C CNN
 F 3 "~" H 11950 2950 50  0001 C CNN
 F 4 "SMD" H 11950 2950 50  0001 C CNN "Soldering"
@@
 	14500 2600 14700 2600
 Text Notes 14700 2250 0    100  ~ 0
-5V OUT\n
+5V/3A OUT\n
 Text Notes 9800 2350 2    100  ~ 0
 9V IN\n
 $Comp
-L EH-900:R R318
+L EH-900-rescue:R-EH-900 R318
 U 1 1 625D065F
 P 12400 2950
 F 0 "R318" V 12300 2850 50  0000 L CNN
 F 1 "20k/THICK" V 12500 2850 50  0000 L CNN
-F 2 "Resistor_SMD:R_0402_1005Metric_Pad0.72x0.64mm_HandSolder" V 12330 2950 50  0001 C CNN
+F 2 "Resistor_SMD:R_0603_1608Metric_Pad0.98x0.95mm_HandSolder" V 12330 2950 50  0001 C CNN
 F 3 "~" H 12400 2950 50  0001 C CNN
 F 4 "SMD" H 12400 2950 50  0001 C CNN "Soldering"
@@
 	11750 2600 11750 2950
 $Comp
-L EH-900:C C311
+L EH-900-rescue:C-EH-900 C311
 U 1 1 625FB292
 P 12600 3450
@@
 5-6 SHORT=ON\n
 $Comp
-L main-eagle-import:DF11-6DP-2DSA CN302
+L EH-900-rescue:DF11-6DP-2DSA-main-eagle-import CN302
 U 1 1 62616009
 P 9750 2900
@@
 	10100 3450 12200 3450
 $Comp
-L EH-900:DF11-4DP-2DSA CN301
+L EH-900-rescue:DF11-4DP-2DSA-EH-900 CN301
 U 1 1 626593A7
 P 8750 2750
@@
 	1    0    0    -1
 $EndComp
+Wire Wire Line
+	8150 2600 8150 3850
+Wire Wire Line
+	8150 3850 5600 3850
+Wire Wire Line
+	5600 3850 5600 4200
+Connection ~ 8150 2600
+Wire Wire Line
+	8150 2600 8550 2600
+Text Label 3750 2900 0    50   ~ 0
+CC1
+Text Label 3750 3000 0    50   ~ 0
+CC2
 $EndSCHEMATC
