File: measurement_unit.sch (KiCad schematic (older format))
At the start: 63 parts, among them CN401 DF11-4DP-2DSA, CN402 DF11-8DP-2DSA, CN403 5267-06A, Q401 SSM3K15AFU, U401 OPA2344EA, U402 MB85RC256V, U403 ADS1115IDGS, U404 TPS79933DDC, U405 DAC80501ZDGS, U406 MCP4725A0T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

Commit message: Rev.01-Add USB-PD CKT
Parts:
- C401, C403, C404, C405, C411, C412, C413: symbol EH-900:C -> EH-900-rescue:C-EH-900
- CN401: symbol EH-900:DF11-4DP-2DSA -> EH-900-rescue:DF11-4DP-2DSA-EH-900
- CN402: symbol EH-900:DF11-8DP-2DSA -> EH-900-rescue:DF11-8DP-2DSA-EH-900
- CN403: symbol EH-900:HNC2-2.5P-6DS -> EH-900-rescue:HNC2-2.5P-6DS-EH-900
- D403: symbol EH-900:1SS -> EH-900-rescue:1SS-EH-900
- L401, L402: symbol EH-900:CommonModeChork_1423 -> EH-900-rescue:CommonModeChork_1423-EH-900
- Q401: symbol EH-900:Q_NMOS_DGS -> EH-900-rescue:Q_NMOS_DGS-EH-900
- R401, R403, R405, R406, R407, R408, R409, R410, R415, R416, R419, R421, R426, R427, R428, R429: symbol EH-900:R -> EH-900-rescue:R-EH-900
- R402, R404: value 10k -> 100k/THICK; symbol EH-900:R -> EH-900-rescue:R-EH-900
- R411, R412, R413, R414, R417, R418, R420, R422, R423, R424, R425, R430, R431: symbol EH-900:R_Thick_1608_Pban -> EH-900-rescue:R_Thick_1608_Pban-EH-900
- U401: symbol ET_OPAMP_STD:OPA2344EA -> EH-900-rescue:OPA2344EA-ET_OPAMP_STD
- U402: symbol EH-900:MB85RC256V -> EH-900-rescue:MB85RC256V-EH-900
- U403: symbol EH-900:ADS1115IDGS -> EH-900-rescue:ADS1115IDGS-EH-900
- U404: symbol EH-900:TPS79933DDC -> EH-900-rescue:TPS79933DDC-EH-900
- U405: symbol EH-900:DAC80501ZDGS -> EH-900-rescue:DAC80501ZDGS-EH-900
- U406: symbol EH-900:MCP4725A0T -> EH-900-rescue:MCP4725A0T-EH-900
- U409: symbol EH-900:LT3922 -> EH-900-rescue:LT3922-EH-900
